Commit message: Create link and joint camera

File: buddy_description/urdf/buddy_description.urdf (robot description, URDF)
Before this commit: robot buddy_description, 14 links, 13 joints
Links:
- added link camera_link; collision box size=0.015 0.030 0.027
Joints:
- added joint camera_joint: type fixed, parent base_link, child camera_link, origin xyz=0.0 -0.05 0.4 rpy=0 0 0

Commit message: Delete camera collision for problems with MoveIt

File: buddy_description/urdf/buddy_description.urdf (robot description, URDF)
Before this commit: robot buddy_description, 15 links, 14 joints
Links:
- link camera_link: geometry 

Commit message: Update joint camera

File: buddy_description/urdf/buddy_description.urdf (robot description, URDF)
Before this commit: robot buddy_description, 15 links, 14 joints
Joints:
- joint camera_joint: origin xyz=0.0 -0.05 0.4 rpy=0 0 0 -> xyz=0.07 0.17 0.0 rpy=0 0 0; parent base_link -> link_4

Commit message: Update urdf for axis rotation

File: buddy_description/urdf/buddy_description.urdf (robot description, URDF)
Before this commit: robot buddy_description, 15 links, 14 joints
Joints:
- joint joint_11: axis -1 0 0 -> 1 0 0
- joint joint_7: axis -1 0 0 -> 1 0 0
- joint joint_9: axis 1 0 0 -> -1 0 0
