Commit message: Corregir alto inicial en simulacion

File: coco_description/urdf/coco_description_sim.xacro.urdf (robot description, URDF)
Before this commit: robot coco_description_sim, 15 links, 14 joints
Joints:
- joint base_joint: origin xyz=0.0 0.0 0.15 rpy=0 0 0.0 -> xyz=0.0 0.0 0.25 rpy=0 0 0.0
