Commit message: Update axis rotation for joint 9

File: coco_description/urdf/coco_description.urdf (robot description, URDF)
Before this commit: robot coco_description, 15 links, 14 joints
Joints:
- joint joint_9: axis -1 0 0 -> 1 0 0

File: coco_description/urdf/coco_description_moveit.urdf (robot description, URDF)
Before this commit: robot coco_description, 15 links, 14 joints
Joints:
- joint joint_9: axis -1 0 0 -> 1 0 0

File: coco_description/urdf/coco_description_sim.xacro.urdf (robot description, URDF)
Before this commit: robot coco_description_sim, 15 links, 14 joints
Joints:
- joint joint_6: limit lower=0 upper=1.0472 effort=300 velocity=3 -> lower=0.000 upper=1.0472 effort=300 velocity=3
- joint joint_9: axis -1 0 0 -> 1 0 0
