Commit message: New urdf for moveit2

File: coco_moveit2_config/config/coco_description.urdf.xacro (robot description, xacro)
@@ -3,7 +3,7 @@
     <xacro:arg name="initial_positions_file" default="initial_positions.yaml" />
     <!-- Import coco_description urdf file -->
-    <xacro:include filename="$(find coco_description)/urdf/coco_description.urdf" />
+    <xacro:include filename="$(find coco_description)/urdf/coco_description_moveit.urdf" />
     <!-- Import control_xacro -->
-    <xacro:include filename="coco_description.ros2_control.xacro" />
-    <xacro:coco_description_ros2_control name="FakeSystem" initial_positions_file="$(arg initial_positions_file)"/>
+    <xacro:include filename="coco_description_moveit.ros2_control.xacro" />
+    <xacro:coco_description_moveit_ros2_control name="FakeSystem" initial_positions_file="$(arg initial_positions_file)"/>
 </robot>

File: coco_moveit2_config/config/coco_description_moveit.ros2_control.xacro (robot description, xacro)
@@ -1,5 +1,5 @@
 <?xml version="1.0"?>
 <robot xmlns:xacro="http://www.ros.org/wiki/xacro">
-    <xacro:macro name="coco_description_ros2_control" params="name initial_positions_file">
+    <xacro:macro name="coco_description_moveit_ros2_control" params="name initial_positions_file">
         <xacro:property name="initial_positions" value="${load_yaml(initial_positions_file)['initial_positions']}"/>
         <ros2_control name="${name}" type="system">
